File: PCB/The Operator.kicad_pcb (KiCad board)
At the start: 2 copper layers, 107 x 67 mm, 24 parts, among them SW1 SW_Push, SW2 SW_Push, SW3 SW_Push, SW4 SW_Push, SW5 RotaryEncoder_Switch, U1 MOUDLE-SEEEDUINO-XIAO

Commit message: fixed leds
Parts:
- D1, D10, D11, D12, D13, D14, D15, D16, D2, D3, D4, D5, D6, D7, D8, D9: value WS2812B -> SK6812MINI-E; footprint LED_SMD:LED_WS2812B_PLCC4_5.0x5.0mm_P3.2mm -> footprints:SK6812MINI-E_fixed
- moved D1 64.4 mm to (101.0, 130.0)
- moved D10 59.7 mm to (145.5, 72.5)
- moved D3 59.3 mm to (129.9, 130.0)
- moved D11 59.3 mm to (129.5, 72.5)
- moved D12 59.2 mm to (113.7, 72.5)
- moved D2 56.5 mm to (115.0, 130.0)
- moved D9 52.8 mm to (183.6, 94.5)
- moved D4 52.8 mm to (143.5, 130.0)
- moved D13 50.6 mm to (99.5, 72.7)
- moved D16 47.6 mm to (88.0, 119.0)
- moved D5 34.4 mm to (157.0, 130.0)
- moved D8 32.7 mm to (183.5, 109.5)
- moved D15 20.8 mm to (88.0, 102.2)
- moved D14 17.1 mm to (88.0, 83.5)
- moved D6 14.0 mm to (172.5, 130.0)
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Routing:
- net Net-(D3-DOUT): track 111.4 -> 27.0 mm, vias 2 -> 0
- net Net-(D10-DIN): track 12.6 -> 54.6 mm, vias 2 -> 0
- net EC11A: track 82.0 -> 41.1 mm, vias 1 -> 0
- net Net-(D13-DOUT): track 43.3 -> 11.9 mm, vias 2 -> 0
- net VCC: track 294.6 -> 323.9 mm, vias 2 -> 13
- net Net-(D6-DOUT): track 7.98 -> 29.6 mm, vias 0 -> 2
- net SCL: track 122.7 -> 141.2 mm, vias 1 -> 0
- net GND: track 469.9 -> 452.5 mm, vias 15 -> 19
- net Net-(D15-DOUT): track 34.0 -> 17.4 mm, vias 2 -> 0
- net Net-(D1-DOUT): track 15.0 -> 30.1 mm
- net Net-(D8-DOUT): track 12.0 -> 25.3 mm, vias 2 -> 0
- net Net-(D12-DOUT): track 21.9 -> 9.61 mm, vias 2 -> 0
- net Net-(D5-DOUT): track 15.8 -> 26.2 mm, vias 2 -> 0
- net Net-(D2-DOUT): track 39.3 -> 29.1 mm
- net Net-(D4-DOUT): track 16.3 -> 26.1 mm, vias 2 -> 0
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
Commit message: fixed oled
Parts:
- moved Brd1 7.50 mm to (95.0, 91.5), turned to 180 degrees
Routing:
- net SCL: track 141.2 -> 80.9 mm
- net SDA: track 106.0 -> 85.4 mm, vias 5 -> 0
- net GND: track 452.5 -> 444.7 mm, vias 19 -> 18
- net VCC: track 323.9 -> 318.8 mm
